File: kicad_proj/mte_usb_hub/mte_usb_hub.kicad_pcb (KiCad board)
At the start: 0 parts

Commit message: New changes from the livestream
Starts the layout
Parts:
- added C1: CC0402KRX5R7BB104, mte_usb_footprints:CAPACITOR_0402N, F.Cu at (114.5, 56.9)
- added C10: CC0402KRX5R7BB104, mte_usb_footprints:CAPACITOR_0402N, F.Cu at (124.7, 143.6)
- added C11: CC0402KRX5R7BB104, mte_usb_footprints:CAPACITOR_0402N, F.Cu at (116.1, 143.6)
- added C12: CC0402KRX5R7BB104, mte_usb_footprints:CAPACITOR_0402N, F.Cu at (119.0, 147.4)
- added C13: CC0402KRX5R7BB104, mte_usb_footprints:CAPACITOR_0402N, F.Cu at (119.0, 145.5)
- added C14: CC0402KRX5R7BB104, mte_usb_footprints:CAPACITOR_0402N, F.Cu at (121.8, 145.5)
- added C15: CC0402KRX5R7BB105, mte_usb_footprints:CAPACITOR_0402N, F.Cu at (139.5, 100.9)
- added C16: CC0402KRX5R7BB105, mte_usb_footprints:CAPACITOR_0402N, F.Cu at (130.9, 102.8)
- added C17: CC0402KRX5R7BB105, mte_usb_footprints:CAPACITOR_0402N, F.Cu at (139.5, 106.7)
- added C18: CC0402KRX5R7BB105, mte_usb_footprints:CAPACITOR_0402N, F.Cu at (133.8, 104.7)
- added C19: CC0402KRX5R7BB105, mte_usb_footprints:CAPACITOR_0402N, F.Cu at (139.5, 98.9)
- added C2: CC0402KRX5R7BB104, mte_usb_footprints:CAPACITOR_0402N, F.Cu at (121.8, 143.6)
- added C20: CC0402JRNPO9BN330, mte_usb_footprints:CAPACITOR_0402N, F.Cu at (128.1, 104.7)
- added C21: CC0402JRNPO9BN270, mte_usb_footprints:CAPACITOR_0402N, F.Cu at (139.5, 104.7)
- added C22: CC0402KRX5R7BB105, mte_usb_footprints:CAPACITOR_0402N, F.Cu at (136.6, 102.8)
- added C23: CC0402JRNPO9BN330, mte_usb_footprints:CAPACITOR_0402N, F.Cu at (133.8, 98.9)
- added C24: CC0402JRNPO9BN270, mte_usb_footprints:CAPACITOR_0402N, F.Cu at (142.3, 98.9)
- added C25: CC0402KRX5R7BB105, mte_usb_footprints:CAPACITOR_0402N, F.Cu at (133.8, 110.5)
- added C26: CC0402KRX5R7BB105, mte_usb_footprints:CAPACITOR_0402N, F.Cu at (142.3, 102.8)
- added C27: CC0402KRX5R7BB105, mte_usb_footprints:CAPACITOR_0402N, F.Cu at (133.8, 108.6)
- added C28: CC0402KRX5R7BB105, mte_usb_footprints:CAPACITOR_0402N, F.Cu at (124.8, 114.9)
- added C29: CC0402KRX5R7BB105, mte_usb_footprints:CAPACITOR_0402N, F.Cu at (136.6, 108.6)
- added C3: CC0402KRX5R7BB104, mte_usb_footprints:CAPACITOR_0402N, F.Cu at (113.3, 147.4)
- added C30: CC0402KRX5R7BB105, mte_usb_footprints:CAPACITOR_0402N, F.Cu at (136.6, 104.7)
- added C31: CC0402KRX5R7BB105, mte_usb_footprints:CAPACITOR_0402N, F.Cu at (130.9, 98.9)
- added C32: CC0402KRX5R7BB105, mte_usb_footprints:CAPACITOR_0402N, F.Cu at (136.6, 98.9)
- added C33: CC0402KRX5R7BB105, mte_usb_footprints:CAPACITOR_0402N, F.Cu at (130.5, 112.5)
- added C34: CC0402KRX5R7BB105, mte_usb_footprints:CAPACITOR_0402N, F.Cu at (142.3, 100.9)
- added C35: CC0402KRX5R7BB105, mte_usb_footprints:CAPACITOR_0402N, F.Cu at (127.7, 113.0)
- added C36: CC0402KRX5R7BB105, mte_usb_footprints:CAPACITOR_0402N, F.Cu at (128.1, 98.9)
- added C37: CC0402KRX5R7BB105, mte_usb_footprints:CAPACITOR_0402N, F.Cu at (139.7, 123.5)
- added C38: CC0402KRX5R7BB105, mte_usb_footprints:CAPACITOR_0402N, F.Cu at (132.4, 130.0)
- added C39: CC0402KRX5R7BB105, mte_usb_footprints:CAPACITOR_0402N, F.Cu at (135.2, 128.1)
- added C4: CC0402KRX5R7BB104, mte_usb_footprints:CAPACITOR_0402N, F.Cu at (129.3, 139.9)
- added C40: CC0402KRX5R7BB105, mte_usb_footprints:CAPACITOR_0402N, F.Cu at (136.8, 121.6)
- added C41: CC0603KRX5R9BB105, mte_usb_footprints:CAPACITOR_0603N, F.Cu at (88.0, 54.5)
- added C42: CC0603KRX5R9BB105, mte_usb_footprints:CAPACITOR_0603N, F.Cu at (88.3, 70.5)
- added C43: GCJ32EC71E226KE02, mte_usb_footprints:CAPACITOR_1210N, F.Cu at (87.6, 76.2)
- added C44: GCJ32EC71E226KE02, mte_usb_footprints:CAPACITOR_1210N, F.Cu at (87.6, 79.5)
- added C45: GCJ32EC71E226KE02, mte_usb_footprints:CAPACITOR_1210N, F.Cu at (79.8, 83.5)
- added C46: EEE-HAE471UAP, mte_usb_footprints:CAPAE1030X1080L350X120N, F.Cu at (36.4, 55.9)
- added C47: EEE-HAE471UAP, mte_usb_footprints:CAPAE1030X1080L350X120N, F.Cu at (87.8, 94.8)
- added C48: GCJ32EC71E226KE02, mte_usb_footprints:CAPACITOR_1210N, F.Cu at (87.6, 73.0)
- added C49: GRM31CR71E106KA12L, mte_usb_footprints:CAPACITOR_1206N, F.Cu at (182.0, 66.4)
- added C5: CC0402KRX5R7BB104, mte_usb_footprints:CAPACITOR_0402N, F.Cu at (116.1, 145.5)
- added C50: GRM31CR71E106KA12L, mte_usb_footprints:CAPACITOR_1206N, F.Cu at (187.5, 63.2)
- added C51: GRM31CR71E106KA12L, mte_usb_footprints:CAPACITOR_1206N, F.Cu at (182.0, 63.2)
- added C52: GRM31CR71E106KA12L, mte_usb_footprints:CAPACITOR_1206N, F.Cu at (188.6, 57.5)
- added C53: CC0402KRX5R7BB104, mte_usb_footprints:CAPACITOR_0402N, F.Cu at (191.7, 62.0)
- added C54: CL21A226MOCLRNC, mte_usb_footprints:CAPACITOR_0805N, F.Cu at (193.4, 57.3)
- added C55: CL21A226MOCLRNC, mte_usb_footprints:CAPACITOR_0805N, F.Cu at (181.3, 69.5)
- added C56: GRM31CR71E106KA12L, mte_usb_footprints:CAPACITOR_1206N, F.Cu at (48.2, 61.7)
- added C57: GRM31CR71E106KA12L, mte_usb_footprints:CAPACITOR_1206N, F.Cu at (50.6, 61.7)
- added C58: GRM31CR71E106KA12L, mte_usb_footprints:CAPACITOR_1206N, F.Cu at (44.7, 60.2)
- added C59: GRM31CR71E106KA12L, mte_usb_footprints:CAPACITOR_1206N, F.Cu at (44.7, 62.4)
- added C6: CC0402KRX5R7BB104, mte_usb_footprints:CAPACITOR_0402N, F.Cu at (113.3, 145.5)
- added C60: GRM31CR71E106KA12L, mte_usb_footprints:CAPACITOR_1206N, F.Cu at (44.7, 64.7)
- added C61: CC0402KRX5R7BB104, mte_usb_footprints:CAPACITOR_0402N, F.Cu at (134.3, 80.3)
- added C62: TMK105BJ153KV-F, mte_usb_footprints:CAPACITOR_0402N, F.Cu at (30.0, 69.9)
- added C63: TMK105ABJ474KV-F, mte_usb_footprints:CAPACITOR_0402N, F.Cu at (39.2, 68.2)
- added C64: TMK105CBJ225MV-F, mte_usb_footprints:CAPACITOR_0402N, F.Cu at (30.0, 65.8)
- added C65: C0402C121J3GAC7867, mte_usb_footprints:CAPACITOR_0402N, F.Cu at (40.0, 62.7)
- added C66: GRM32ER60J227ME05L, mte_usb_footprints:CAPACITOR_1210N, F.Cu at (40.7, 90.2)
- added C67: GRM32ER60J227ME05L, mte_usb_footprints:CAPACITOR_1210N, F.Cu at (40.7, 93.6)
- added C68: GRM32ER60J227ME05L, mte_usb_footprints:CAPACITOR_1210N, F.Cu at (40.7, 97.0)
- added C69: CC0402KRX5R7BB105, mte_usb_footprints:CAPACITOR_0402N, F.Cu at (208.7, 56.9)
- added C7: CC0402KRX5R7BB104, mte_usb_footprints:CAPACITOR_0402N, F.Cu at (113.3, 143.6)
- added C70: CC0402KRX5R7BB105, mte_usb_footprints:CAPACITOR_0402N, F.Cu at (208.7, 58.8)
- added C71: GRM21BR61H106ME43, mte_usb_footprints:CAPACITOR_0805N, F.Cu at (170.7, 98.8)
- added C72: GRM21BR61H106ME43, mte_usb_footprints:CAPACITOR_0805N, F.Cu at (175.4, 94.0)
- added C73: GRM21BR61H106ME43, mte_usb_footprints:CAPACITOR_0805N, F.Cu at (152.7, 88.3)
- added C74: GRM21BR61H106ME43, mte_usb_footprints:CAPACITOR_0805N, F.Cu at (157.2, 82.2)
- added C75: TMK105CBJ225MV-F, mte_usb_footprints:CAPACITOR_0402N, F.Cu at (75.6, 54.6)
- added C76: TMK105CBJ225MV-F, mte_usb_footprints:CAPACITOR_0402N, F.Cu at (80.2, 51.5)
- added C77: GRM21BR61H106ME43, mte_usb_footprints:CAPACITOR_0805N, F.Cu at (151.1, 126.8)
- added C78: GRM21BR61H106ME43, mte_usb_footprints:CAPACITOR_0805N, F.Cu at (155.9, 122.1)
- added C79: GRM21BR61H106ME43, mte_usb_footprints:CAPACITOR_0805N, F.Cu at (199.4, 81.8)
- added C8: CC0402KRX5R7BB104, mte_usb_footprints:CAPACITOR_0402N, F.Cu at (116.1, 147.4)
- added C80: GRM21BR61H106ME43, mte_usb_footprints:CAPACITOR_0805N, F.Cu at (203.9, 75.7)
- added C81: GRM21BR61H106ME43, mte_usb_footprints:CAPACITOR_0805N, F.Cu at (114.7, 128.2)
- added C82: GRM21BR61H106ME43, mte_usb_footprints:CAPACITOR_0805N, F.Cu at (119.2, 122.1)
- added C83: GRM21BR61H106ME43, mte_usb_footprints:CAPACITOR_0805N, F.Cu at (152.7, 106.7)
- added C84: GRM21BR61H106ME43, mte_usb_footprints:CAPACITOR_0805N, F.Cu at (157.2, 100.5)
- added C9: CC0402KRX5R7BB104, mte_usb_footprints:CAPACITOR_0402N, F.Cu at (119.0, 143.6)
- added D1: BAS16GWJ, mte_usb_footprints:SODFL360X160X130L45X62N, F.Cu at (201.9, 66.7)
- added D10: ESD8004MUTAG, mte_usb_footprints:ESD8004MUTAG, F.Cu at (47.0, 148.0)
- added D11: ESD9X3.3ST5G, mte_usb_footprints:SODFL1006X43N, F.Cu at (203.2, 78.1)
- added D12: ESD8004MUTAG, mte_usb_footprints:ESD8004MUTAG, F.Cu at (37.0, 148.0)
- added D13: ESD8004MUTAG, mte_usb_footprints:ESD8004MUTAG, F.Cu at (31.0, 148.0)
- added D14: ESD9X3.3ST5G, mte_usb_footprints:SODFL1006X43N, F.Cu at (118.6, 124.5)
- added D15: ESD8004MUTAG, mte_usb_footprints:ESD8004MUTAG, F.Cu at (86.4, 148.0)
- added D16: ESD8004MUTAG, mte_usb_footprints:ESD8004MUTAG, F.Cu at (81.0, 148.0)
- added D17: ESD9X3.3ST5G, mte_usb_footprints:SODFL1006X43N, F.Cu at (156.5, 103.0)
- added D2: ESD8004MUTAG, mte_usb_footprints:ESD8004MUTAG, F.Cu at (69.4, 148.0)
- added D3: ESD8004MUTAG, mte_usb_footprints:ESD8004MUTAG, F.Cu at (64.0, 148.0)
- added D4: ESD9X3.3ST5G, mte_usb_footprints:SODFL1006X43N, F.Cu at (156.5, 84.6)
- added D5: ESD8004MUTAG, mte_usb_footprints:ESD8004MUTAG, F.Cu at (64.4, 60.4)
- added D6: ESD8004MUTAG, mte_usb_footprints:ESD8004MUTAG, F.Cu at (56.8, 60.4)
- added D7: ESD8004MUTAG, mte_usb_footprints:ESD8004MUTAG, F.Cu at (60.6, 60.4)
- added D8: ESD9X3.3ST5G, mte_usb_footprints:SODFL1006X43N, F.Cu at (71.0, 57.7)
- added D9: ESD8004MUTAG, mte_usb_footprints:ESD8004MUTAG, F.Cu at (52.4, 148.0)
- added J1: Conn_01x02_Male, Connector_PinHeader_2.54mm:PinHeader_1x02_P2.54mm_Vertical, F.Cu at (89.3, 51.8)
- added J2: USB_C_Receptacle, Connector_USB:USB_C_Receptacle_Amphenol_12401610E4-2A, F.Cu at (60.8, 53.2)
- added J3: USB3_A, Connector_USB:USB3_A_Molex_48393-001, F.Cu at (32.5, 152.8)
- added J4: USB3_A, Connector_USB:USB3_A_Molex_48393-001, F.Cu at (82.9, 152.8)
- added J5: USB3_A, Connector_USB:USB3_A_Molex_48393-001, F.Cu at (65.9, 152.8)
- added J6: USB3_A, Connector_USB:USB3_A_Molex_48393-001, F.Cu at (48.9, 152.8)
- added L1: ACM1211-701-2PL-TL01, mte_usb_footprints:ACM1211-701-2PL-TL01, F.Cu at (88.3, 62.5)
- added L2: FCUL0624-H-R22M=P3, mte_usb_footprints:INDM730X660X240L150X140N, F.Cu at (86.0, 85.0)
- added L3: 74405042022, mte_usb_footprints:INDM400X400X200L95X310N, F.Cu at (182.5, 58.7)
- added L4: SRP1270-1R5M, mte_usb_footprints:INDM1350X1350X700L250X300N, F.Cu at (39.2, 80.7)
- added Q1: CSD16342Q5A, mte_usb_footprints:CSD16342Q5A, F.Cu at (47.3, 69.2)
- added Q2: CSD17577Q5AT, mte_usb_footprints:CSD16342Q5A, F.Cu at (42.3, 69.2)
- added R1: RC0402JR-0710KL, mte_usb_footprints:RESISTOR_0402N, F.Cu at (130.5, 114.4)
- added R10: RC0402JR-0747KL, mte_usb_footprints:RESISTOR_0402N, F.Cu at (133.8, 106.7)
- added R11: RC0402JR-0710KL, mte_usb_footprints:RESISTOR_0402N, F.Cu at (133.8, 100.9)
- added R12: RC0402JR-07200KL, mte_usb_footprints:RESISTOR_0402N, F.Cu at (128.1, 106.7)
- added R13: RC0402JR-07200KL, mte_usb_footprints:RESISTOR_0402N, F.Cu at (127.7, 114.9)
- added R14: RC0402JR-07200KL, mte_usb_footprints:RESISTOR_0402N, F.Cu at (122.0, 114.9)
- added R15: RC0402JR-0710RL, mte_usb_footprints:RESISTOR_0402N, F.Cu at (133.8, 102.8)
- added R16: RC0402JR-0747KL, mte_usb_footprints:RESISTOR_0402N, F.Cu at (119.1, 114.9)
- added R17: RC0402JR-0747KL, mte_usb_footprints:RESISTOR_0402N, F.Cu at (145.2, 98.9)
- added R18: RC0402JR-0747KL, mte_usb_footprints:RESISTOR_0402N, F.Cu at (130.9, 104.7)
- added R19: RC0402JR-0747KL, mte_usb_footprints:RESISTOR_0402N, F.Cu at (130.9, 110.5)
- added R2: RC0402JR-0747KL, mte_usb_footprints:RESISTOR_0402N, F.Cu at (119.1, 113.0)
- added R20: RC0402JR-0710KL, mte_usb_footprints:RESISTOR_0402N, F.Cu at (128.1, 110.5)
- added R21: RC0402JR-0710KL, mte_usb_footprints:RESISTOR_0402N, F.Cu at (128.1, 102.8)
- added R22: RC0402JR-0710KL, mte_usb_footprints:RESISTOR_0402N, F.Cu at (130.9, 100.9)
- added R23: RT0402DRE0712KL, mte_usb_footprints:RESISTOR_0402N, F.Cu at (136.6, 100.9)
- added R24: RC0402JR-0710KL, mte_usb_footprints:RESISTOR_0402N, F.Cu at (136.6, 106.7)
- added R25: RC0402JR-0710KL, mte_usb_footprints:RESISTOR_0402N, F.Cu at (122.0, 113.0)
- added R26: RC0402FR-07887KL, mte_usb_footprints:RESISTOR_0402N, F.Cu at (132.4, 128.1)
- added R27: RC0402JR-07200KL, mte_usb_footprints:RESISTOR_0402N, F.Cu at (136.8, 123.5)
- added R28: RC0402JR-074K7L, mte_usb_footprints:RESISTOR_0402N, F.Cu at (139.7, 121.6)
- added R29: RC0402JR-074K7L, mte_usb_footprints:RESISTOR_0402N, F.Cu at (136.8, 125.5)
- added R3: RC0402JR-0747KL, mte_usb_footprints:RESISTOR_0402N, F.Cu at (139.5, 102.8)
- added R30: RL1206JR-070R51L, mte_usb_footprints:RESISTOR_1206N, F.Cu at (83.8, 74.5)
- added R32: RC0402JR-0710KL, mte_usb_footprints:RESISTOR_0402N, F.Cu at (190.1, 60.1)
- added R33: RC0402JR-0710KL, mte_usb_footprints:RESISTOR_0402N, F.Cu at (187.2, 60.1)
- added R34: RC0402FR-0780K6L, mte_usb_footprints:RESISTOR_0402N, F.Cu at (31.0, 71.6)
- added R35: RC0402FR-071K58L, mte_usb_footprints:RESISTOR_0402N, F.Cu at (37.5, 71.7)
- added R36: RC0402FR-0773K2L, mte_usb_footprints:RESISTOR_0402N, F.Cu at (40.0, 63.7)
- added R37: RC0402JR-0710KL, mte_usb_footprints:RESISTOR_0402N, F.Cu at (38.0, 63.7)
- added R4: RC0402JR-0747KL, mte_usb_footprints:RESISTOR_0402N, F.Cu at (130.9, 108.6)
- added R5: RC0402JR-0747KL, mte_usb_footprints:RESISTOR_0402N, F.Cu at (133.4, 112.5)
- added R6: RC0402JR-0747KL, mte_usb_footprints:RESISTOR_0402N, F.Cu at (128.1, 108.6)
- added R7: RC0402JR-0747KL, mte_usb_footprints:RESISTOR_0402N, F.Cu at (124.8, 113.0)
- added R8: RC0402JR-0747KL, mte_usb_footprints:RESISTOR_0402N, F.Cu at (130.9, 106.7)
- added R9: RC0402JR-0747KL, mte_usb_footprints:RESISTOR_0402N, F.Cu at (128.1, 100.9)
- added R?1: RC0402FR-07390RL, mte_usb_footprints:RESISTOR_0402N, F.Cu at (211.6, 56.9)
- added R?2: RC0402JR-07240RL, mte_usb_footprints:RESISTOR_0402N, F.Cu at (200.6, 69.2)
- added U1: USB7206, mte_usb_footprints:QFN101P40_1200X1200X90L60X20T800N, F.Cu at (61.6, 80.4)
- added U2: HD3SS3220, mte_usb_footprints:QFN31P40_250X450X80L30X20T120X320N, F.Cu at (60.6, 64.8)
- added U3: TPS563207SDRLR, mte_usb_footprints:SOL6P50_160X160X60L21N, F.Cu at (186.3, 66.7)
- added U4: LM3150MH, mte_usb_footprints:SOP15P65_500X640X110L60X24T310X300N, F.Cu at (34.3, 68.2)
- added U5: UCS2114, mte_usb_footprints:UCS2114, F.Cu at (171.1, 95.2)
- added U6: UCS2114, mte_usb_footprints:UCS2114, F.Cu at (151.6, 123.2)
- added U?1: LM317DCYR, mte_usb_footprints:SOT223-4P230_700X180L80X75N, F.Cu at (203.2, 60.5)
- added Y1: RH100-25.000-20-F-1030-TR, mte_usb_footprints:RH100-12.000-10-2020-EXT-TR, F.Cu at (115.1, 114.1)
Routing:
- net +12V: track 0.00 -> 89.5 mm, vias 0 -> 1
- net +5V: track 0.00 -> 65.8 mm, vias 0 -> 4
- net Net-(C42-Pad1): track 0.00 -> 24.0 mm
- net Net-(Q1-Pad4): track 0.00 -> 17.5 mm, vias 0 -> 2
- net Net-(C65-Pad2): track 0.00 -> 12.6 mm
- net /USB2DN_4_DP: track 0.00 -> 12.3 mm
- net Net-(C63-Pad2): track 0.00 -> 10.0 mm
- net /USB2DN_4_DN: track 0.00 -> 9.29 mm
- net GND: track 0.00 -> 8.73 mm
- net /INPUT FILTER/VIN: track 0.00 -> 6.68 mm
- net /INPUT FILTER/GND_IN: track 0.00 -> 6.27 mm
- net /USB3DN_4_RXDP: track 0.00 -> 5.12 mm
- net /USB3DN_4_TXDN: track 0.00 -> 4.98 mm
- net /USB_A Filter_3/USB3_RXDN: track 0.00 -> 4.27 mm
- net /USB3DN_4_TXDP: track 0.00 -> 4.27 mm
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- added copper zone on In3.Cu, net +5V
- added copper zone on F.Cu, net GND
Other:
- board outline added: 69 x 113.2 mm
- copper layers 0 -> 6
