File: kicad_proj/mte_usb_hub/mte_usb_hub.kicad_pcb (KiCad board)
At the start: 6 copper layers, 69 x 113.2 mm, 159 parts, among them J1 Conn_01x02_Male, J2 USB_C_Receptacle, J3 USB3_A, J4 USB3_A, J5 USB3_A, J6 USB3_A, Q1 CSD16342Q5A, Q2 CSD17577Q5AT, U1 USB7206, U2 HD3SS3220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

Commit message: Updates from the livestream
Parts:
- moved C80 185.6 mm to (20.8, 106.0), turned to -90 degrees
- moved D11 182.8 mm to (22.3, 103.8), turned to 180 degrees
- moved C79 178.2 mm to (22.8, 106.0), turned to -90 degrees
- moved C5 142.8 mm to (49.0, 19.4), turned to -90 degrees
- moved C6 141.0 mm to (50.0, 19.4), turned to -90 degrees
- moved C72 130.0 mm to (46.3, 109.0), turned to -90 degrees
- moved U5 129.2 mm to (42.5, 107.7), turned to 90 degrees
- moved C71 122.8 mm to (48.3, 109.0), turned to -90 degrees
- moved C11 107.5 mm to (16.8, 102.5), turned to 180 degrees
- moved C82 106.0 mm to (14.3, 107.5), turned to 90 degrees
- moved D14 104.8 mm to (14.8, 109.8)
- moved C7 104.5 mm to (16.8, 103.5), turned to 180 degrees
- moved C78 103.9 mm to (52.8, 109.0), turned to -90 degrees
- moved C12 102.2 mm to (30.3, 96.6), turned to -90 degrees
- moved C77 102.0 mm to (50.7, 109.0), turned to -90 degrees
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Connections:
- net /UFP_MUX/RXn renamed /RXN
- net /UFP_MUX/RXp renamed /RXP
- net /UFP_MUX/TXn renamed /TXN
- net /UFP_MUX/TXp renamed /TXP
- net /UFP_MUX/USB2_DOWN_n renamed /USB2_DOWN_N
- net /UFP_MUX/USB2_DOWN_p renamed /USB2_DOWN_P
- net /USB_C Filter/CC1 renamed /UFP_MUX/CC1
- net /USB_C Filter/RX1- renamed /UFP_MUX/RX1n
- D12 pad 1: /USB3DN_3_RXDP -> /USB3DN_1_RXDN
- D12 pad 10: /USB3DN_3_RXDP -> /USB3DN_1_RXDN
- D12 pad 2: /USB3DN_3_RXDN -> /USB3DN_1_RXDP
- D12 pad 4: /USB3DN_3_TXDP -> /USB3DN_1_TXDN
- D12 pad 5: /USB3DN_3_TXDN -> /USB3DN_1_TXDP
- D12 pad 6: /USB3DN_3_TXDN -> /USB3DN_1_TXDP
- D12 pad 7: /USB3DN_3_TXDP -> /USB3DN_1_TXDN
- D12 pad 9: /USB3DN_3_RXDN -> /USB3DN_1_RXDP
- D13 pad 4: /USB2DN_3_DP -> /USB2DN_1_DP
- D13 pad 5: /USB2DN_3_DN -> /USB2DN_1_DN
- D13 pad 6: /USB2DN_3_DN -> /USB2DN_1_DN
- D13 pad 7: /USB2DN_3_DP -> /USB2DN_1_DP
- D15 pad 1: /USB3DN_4_RXDP -> /USB3DN_4_RXDN
- D15 pad 10: /USB3DN_4_RXDP -> /USB3DN_4_RXDN
- D15 pad 2: /USB_A Filter_3/USB3_RXDN -> /USB3DN_4_RXDP
- D15 pad 4: /USB3DN_4_TXDP -> /USB3DN_4_TXDN
- D15 pad 5: /USB3DN_4_TXDN -> /USB3DN_4_TXDP
- D15 pad 6: /USB3DN_4_TXDN -> /USB3DN_4_TXDP
- D15 pad 7: /USB3DN_4_TXDP -> /USB3DN_4_TXDN
- D15 pad 9: /USB_A Filter_3/USB3_RXDN -> /USB3DN_4_RXDP
- D2 pad 1: /USB3DN_1_RXDP -> /USB3DN_3_RXDN
- D2 pad 10: /USB3DN_1_RXDP -> /USB3DN_3_RXDN
- D2 pad 2: /USB3DN_1_RXDN -> /USB3DN_3_RXDP
- D2 pad 4: /USB3DN_1_TXDP -> /USB3DN_3_TXDN
- D2 pad 5: /USB3DN_1_TXDN -> /USB3DN_3_TXDP
- D2 pad 6: /USB3DN_1_TXDN -> /USB3DN_3_TXDP
- D2 pad 7: /USB3DN_1_TXDP -> /USB3DN_3_TXDN
- D2 pad 9: /USB3DN_1_RXDN -> /USB3DN_3_RXDP
- D3 pad 4: /USB2DN_1_DP -> /USB2DN_3_DP
- D3 pad 5: /USB2DN_1_DN -> /USB2DN_3_DN
- D3 pad 6: /USB2DN_1_DN -> /USB2DN_3_DN
- D3 pad 7: /USB2DN_1_DP -> /USB2DN_3_DP
- D9 pad 1: /USB3DN_2_RXDP -> /USB3DN_2_RXDN
- D9 pad 10: /USB3DN_2_RXDP -> /USB3DN_2_RXDN
- D9 pad 2: /USB3DN_2_RXDN -> /USB3DN_2_RXDP
- D9 pad 4: /USB3DN_2_TXDP -> /USB3DN_2_TXDN
- D9 pad 5: /USB3DN_2_TXDN -> /USB3DN_2_TXDP
- D9 pad 6: /USB3DN_2_TXDN -> /USB3DN_2_TXDP
- D9 pad 7: /USB3DN_2_TXDP -> /USB3DN_2_TXDN
- D9 pad 9: /USB3DN_2_RXDN -> /USB3DN_2_RXDP
- J3 pad 2: /USB2DN_3_DN -> /USB2DN_1_DN
- J3 pad 3: /USB2DN_3_DP -> /USB2DN_1_DP
- J3 pad 5: /USB3DN_3_RXDN -> /USB3DN_1_RXDN
- J3 pad 6: /USB3DN_3_RXDP -> /USB3DN_1_RXDP
- J3 pad 8: /USB3DN_3_TXDN -> /USB3DN_1_TXDN
- J3 pad 9: /USB3DN_3_TXDP -> /USB3DN_1_TXDP
- J4 pad 5: /USB_A Filter_3/USB3_RXDN -> /USB3DN_4_RXDN
- J5 pad 2: /USB2DN_1_DN -> /USB2DN_3_DN
- J5 pad 3: /USB2DN_1_DP -> /USB2DN_3_DP
- J5 pad 5: /USB3DN_1_RXDN -> /USB3DN_3_RXDN
- J5 pad 6: /USB3DN_1_RXDP -> /USB3DN_3_RXDP
- J5 pad 8: /USB3DN_1_TXDN -> /USB3DN_3_TXDN
- J5 pad 9: /USB3DN_1_TXDP -> /USB3DN_3_TXDP
- U5 pad 4: /VBUS_1 -> /VBUS_3
- U5 pad 5: /VBUS_1 -> /VBUS_3
- U6 pad 4: /VBUS_3 -> /VBUS_1
- U6 pad 5: /VBUS_3 -> /VBUS_1
Routing:
- net /USB2_DOWN_P: track 0.00 -> 68.2 mm
- net /USB2_DOWN_N: track 0.00 -> 67.8 mm
- net /RXP: track 0.00 -> 56.9 mm
- net /RXN: track 0.00 -> 56.9 mm
- net /USB_HUB/USB3UP_TXDN: track 0.00 -> 56.9 mm
- net /USB_HUB/USB3UP_TXDP: track 0.00 -> 56.9 mm
- net /VBUS_3: track 0.00 -> 53.2 mm
- net (no net): track 0.00 -> 47.2 mm
- net /USB3DN_4_RXDN: track 0.00 -> 46.5 mm
- net /USB2DN_4_DN: track 9.29 -> 54.7 mm, vias 0 -> 3
- net /USB3DN_1_RXDP: track 0.00 -> 41.6 mm
- net /USB3DN_1_RXDN: track 0.00 -> 41.6 mm
- net /USB3DN_4_RXDP: track 5.12 -> 46.0 mm
- net /USB_HUB/USB3DN_4_TXDP: track 0.00 -> 40.0 mm, vias 0 -> 3
- net /USB_HUB/USB3DN_4_TXDN: track 0.00 -> 39.8 mm, vias 0 -> 3
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- added copper zone on In3.Cu, net +3V3
- added copper zone on In2.Cu, net /1.15V
Other:
- board size 69 x 113.2 mm -> 100 x 114 mm

Commit message: Updates from the livestream
Parts:
- moved C40 142.6 mm to (31.9, -5.40)
- moved R28 142.6 mm to (31.9, -3.47)
- moved C37 142.6 mm to (34.7, -3.47)
- moved C38 142.6 mm to (34.7, -7.33)
- moved C39 142.6 mm to (37.6, -7.33)
- moved R27 142.6 mm to (34.7, -5.40)
- moved R29 142.6 mm to (37.6, -5.40)
- moved C3 119.0 mm to (61.6, -12.2)
- moved C61 114.9 mm to (14.6, 16.6)
- moved C4 113.3 mm to (46.3, 15.0), turned to -90 degrees
- moved C2 108.4 mm to (45.3, 15.0), turned to -90 degrees
- moved R26 93.5 mm to (56.2, 71.8), turned to 90 degrees
- moved C24 84.0 mm to (109.8, -14.0)
- moved C33 83.6 mm to (44.0, 75.1), turned to 180 degrees
- moved C21 78.8 mm to (112.6, -14.0)
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Connections:
- net /UFP_MUX/CC1 renamed /USB_C Filter/CC1
- net /UFP_MUX/RX1n renamed /RX1_N
- net /UFP_MUX/RX1p renamed /RX1_P
- net /UFP_MUX/TX1n renamed /TX1_N
- net /UFP_MUX/TX1p renamed /TX1_P
- net /UFP_MUX/TX2n renamed /TX2_N
- net /UFP_MUX/TX2p renamed /TX2_P
- net /USB_C Filter/TX1+ renamed /USB_C Filter/_TX1+
- net /USB_C Filter/TX1- renamed /USB_C Filter/_TX1-
- C2 pad 1: /USB_C Filter/TX2+ -> /USB_C Filter/_TX2+
- C23 pad 1: Net-(C20-Pad1) -> Net-(U1-Pad98)
- C4 pad 1: /USB_C Filter/TX2- -> /USB_C Filter/_TX2-
- D6 pad 1: /UFP_MUX/RX2n -> /RX2_P
- D6 pad 10: /UFP_MUX/RX2n -> /RX2_P
- D6 pad 2: /UFP_MUX/RX2p -> /RX2_N
- D6 pad 4: /USB_C Filter/TX2- -> /USB_C Filter/_TX2+
- D6 pad 5: /USB_C Filter/TX2+ -> /USB_C Filter/_TX2-
- D6 pad 6: /USB_C Filter/TX2+ -> /USB_C Filter/_TX2-
- D6 pad 7: /USB_C Filter/TX2- -> /USB_C Filter/_TX2+
- D6 pad 9: /UFP_MUX/RX2p -> /RX2_N
- J2 pad A10: /UFP_MUX/RX2n -> /RX2_N
- J2 pad A11: /UFP_MUX/RX2p -> /RX2_P
- J2 pad B2: /USB_C Filter/TX2+ -> /USB_C Filter/_TX2+
- J2 pad B3: /USB_C Filter/TX2- -> /USB_C Filter/_TX2-
- U2 pad 18: /UFP_MUX/RX2n -> /RX2_N
- U2 pad 19: /UFP_MUX/RX2p -> /RX2_P
Routing:
- net +12V: track 89.5 -> 23.7 mm, vias 1 -> 0
- net /RXP: track 56.9 -> 0.11 mm
- net /RXN: track 56.9 -> 0.11 mm
- net /USB_HUB/USB3UP_TXDN: track 56.9 -> 0.11 mm
- net /USB_HUB/USB3UP_TXDP: track 56.9 -> 0.11 mm
- net (no net): track 47.2 -> 0.00 mm
- net +5V: track 87.1 -> 52.8 mm, vias 4 -> 2
- net /1.15V: track 0.00 -> 19.5 mm, vias 0 -> 9
- net /USB2_DOWN_P: track 68.2 -> 51.3 mm
- net /USB2_DOWN_N: track 67.8 -> 51.4 mm
- net +3V3: track 12.6 -> 27.4 mm, vias 12 -> 9
- net Net-(C20-Pad1): track 0.00 -> 7.44 mm
- net Net-(U1-Pad98): track 0.00 -> 4.78 mm
- net /USB3DN_4_RXDP: track 46.0 -> 50.3 mm
- net /USB3DN_4_RXDN: track 46.5 -> 50.8 mm
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- added copper zone on B.Cu, net GND
- added copper zone on In1.Cu, net GND
- added copper zone on In4.Cu, net GND

Commit message: Livestream updates
Parts:
- moved C69 90.2 mm to (28.5, 52.2)
- moved C70 90.2 mm to (31.4, 52.2)
- moved D1 90.2 mm to (29.9, 49.7)
- moved R?1 90.2 mm to (28.5, 54.1)
- moved R?2 90.2 mm to (34.0, 49.2)
- moved U?1 90.2 mm to (23.0, 52.8)
- moved C46 81.4 mm to (6.75, 86.0), turned to -90 degrees
- moved C64 74.8 mm to (14.9, 91.3), turned to 180 degrees
- moved C61 74.3 mm to (13.4, 90.9), turned to 90 degrees
- moved C3 74.2 mm to (50.9, 61.2), turned to -90 degrees
- moved C40 74.1 mm to (51.5, 66.0), turned to 180 degrees
- moved C39 73.7 mm to (51.5, 65.0), turned to 180 degrees
- moved C38 73.7 mm to (43.3, 65.8), turned to 90 degrees
- moved R27 73.4 mm to (53.6, 65.5), turned to -90 degrees
- moved C62 70.7 mm to (19.1, 91.3), turned to 0 degrees
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Connections:
- net /USB_C Filter/CC1 renamed /UFP_MUX/CC1
- D10 pad 1: Net-(D10-Pad1) -> unconnected-(D10-Pad1)
- D10 pad 10: Net-(D10-Pad1) -> unconnected-(D10-Pad1)
- D10 pad 2: Net-(D10-Pad2) -> unconnected-(D10-Pad2)
- D10 pad 9: Net-(D10-Pad2) -> unconnected-(D10-Pad2)
- D13 pad 1: Net-(D13-Pad1) -> unconnected-(D13-Pad1)
- D13 pad 10: Net-(D13-Pad1) -> unconnected-(D13-Pad1)
- D13 pad 2: Net-(D13-Pad2) -> unconnected-(D13-Pad2)
- D13 pad 9: Net-(D13-Pad2) -> unconnected-(D13-Pad2)
- D16 pad 1: Net-(D16-Pad1) -> unconnected-(D16-Pad1)
- D16 pad 10: Net-(D16-Pad1) -> unconnected-(D16-Pad1)
- D16 pad 2: Net-(D16-Pad2) -> unconnected-(D16-Pad2)
- D16 pad 9: Net-(D16-Pad2) -> unconnected-(D16-Pad2)
- D3 pad 1: Net-(D3-Pad1) -> unconnected-(D3-Pad1)
- D3 pad 10: Net-(D3-Pad1) -> unconnected-(D3-Pad1)
- D3 pad 2: Net-(D3-Pad2) -> unconnected-(D3-Pad2)
- D3 pad 9: Net-(D3-Pad2) -> unconnected-(D3-Pad2)
- D5 pad 1: /USB_C Filter/_TX1+ -> /USB_C Filter/_TX1-
- D5 pad 10: /USB_C Filter/_TX1+ -> /USB_C Filter/_TX1-
- D5 pad 2: /USB_C Filter/_TX1- -> /USB_C Filter/_TX1+
- D5 pad 9: /USB_C Filter/_TX1- -> /USB_C Filter/_TX1+
- D6 pad 1: /RX2_P -> /USB_C Filter/_TX2+
- D6 pad 10: /RX2_P -> /USB_C Filter/_TX2+
- D6 pad 2: /RX2_N -> /USB_C Filter/_TX2-
- D6 pad 4: /USB_C Filter/_TX2+ -> /RX2_P
- D6 pad 5: /USB_C Filter/_TX2- -> /RX2_N
- D6 pad 6: /USB_C Filter/_TX2- -> /RX2_N
- D6 pad 7: /USB_C Filter/_TX2+ -> /RX2_P
- D6 pad 9: /RX2_N -> /USB_C Filter/_TX2-
- D7 pad 4: /USB2_DOWN_P -> /USB2_DOWN_N
- D7 pad 5: /USB2_DOWN_N -> /USB2_DOWN_P
- D7 pad 6: /USB2_DOWN_N -> /USB2_DOWN_P
- D7 pad 7: /USB2_DOWN_P -> /USB2_DOWN_N
Routing:
- net +12V: track 23.7 -> 87.4 mm, vias 0 -> 4
- net /5V_UFP: track 0.00 -> 40.6 mm
- net /USB2DN_1_DN: track 37.5 -> 0.00 mm
- net /USB2DN_1_DP: track 37.5 -> 0.04 mm
- net /USB2_DOWN_N: track 51.4 -> 23.8 mm, vias 0 -> 2
- net /USB2_DOWN_P: track 51.3 -> 24.9 mm, vias 0 -> 4
- net /UFP_MUX/CC2: track 0.00 -> 20.1 mm, vias 0 -> 7
- net /RX1_N: track 0.00 -> 18.9 mm
- net /RX1_P: track 0.00 -> 17.6 mm
- net /UFP_MUX/CC1: track 0.00 -> 16.7 mm, vias 0 -> 4
- net /RXN: track 0.11 -> 11.7 mm, vias 0 -> 2
- net /RXP: track 0.11 -> 11.0 mm, vias 0 -> 2
- net /RX2_N: track 0.00 -> 10.5 mm
- net /RX2_P: track 0.00 -> 10.5 mm
- net Net-(R26-Pad2): track 0.00 -> 9.09 mm
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Other:
- board text added: "DO NOT PLACE"
