File: kicad_proj/mte_usb_hub/mte_usb_hub.kicad_sch (KiCad schematic)
At the start: 20 parts, among them J1 Conn_01x02_Male, J2 USB_C_Receptacle, J3 USB3_A, J4 USB3_A, J5 USB3_A, J6 USB3_A

Commit message: New changes from the livestream
Starts the layout
Parts:
- C1, C10, C11, C12, C13, C14, C2, C3, C4, C5, C6, C7, C8, C9: footprint footprints:CAPACITOR_0402N -> mte_usb_footprints:CAPACITOR_0402N
- J1: footprint (none) -> Connector_PinHeader_2.54mm:PinHeader_1x02_P2.54mm_Vertical
- J2: footprint (none) -> Connector_USB:USB_C_Receptacle_Amphenol_12401610E4-2A
- J3, J4, J5, J6: footprint (none) -> Connector_USB:USB3_A_Molex_48393-001
Connections:
- net USB_A Filter/USB3_DN_RXDN_OUT: now also J5.5 (SSRX-); no longer J5.8 (SSTX-)
- net USB_A Filter/USB3_DN_RXDP_OUT: now also J5.6 (SSRX+); no longer J5.9 (SSTX+)
- net USB_A Filter/USB3_DN_TXDN_OUT: now also J5.8 (SSTX-); no longer J5.5 (SSRX-)
- net USB_A Filter/USB3_DN_TXDP_OUT: now also J5.9 (SSTX+); no longer J5.6 (SSRX+)
- net USB_A Filter_1/USB3_DN_RXDN_OUT: now also J6.5 (SSRX-); no longer J6.8 (SSTX-)
- net USB_A Filter_1/USB3_DN_RXDP_OUT: now also J6.6 (SSRX+); no longer J6.9 (SSTX+)
- net USB_A Filter_1/USB3_DN_TXDN_OUT: now also J6.8 (SSTX-); no longer J6.5 (SSRX-)
- net USB_A Filter_1/USB3_DN_TXDP_OUT: now also J6.9 (SSTX+); no longer J6.6 (SSRX+)
- net USB_A Filter_2/USB3_DN_RXDN_OUT: now also J3.5 (SSRX-); no longer J3.8 (SSTX-)
- net USB_A Filter_2/USB3_DN_RXDP_OUT: now also J3.6 (SSRX+); no longer J3.9 (SSTX+)
- net USB_A Filter_2/USB3_DN_TXDN_OUT: now also J3.8 (SSTX-); no longer J3.5 (SSRX-)
- net USB_A Filter_2/USB3_DN_TXDP_OUT: now also J3.9 (SSTX+); no longer J3.6 (SSRX+)
- net USB_A Filter_3/USB3_DN_RXDN_OUT: now also J4.5 (SSRX-); no longer J4.8 (SSTX-)
- net USB_A Filter_3/USB3_DN_RXDP_OUT: now also J4.6 (SSRX+); no longer J4.9 (SSTX+)
- net USB_A Filter_3/USB3_DN_TXDN_OUT: now also J4.8 (SSTX-); no longer J4.5 (SSRX-)
- net USB_A Filter_3/USB3_DN_TXDP_OUT: now also J4.9 (SSTX+); no longer J4.6 (SSRX+)
- net USB_HUB/USB3DN_1_TXDM renamed USB_HUB/USB3DN_1_TXDN
- net USB_HUB/USB3DN_2_TXDM renamed USB_HUB/USB3DN_2_TXDN
- net USB_HUB/USB3DN_3_TXDM renamed USB_HUB/USB3DN_3_TXDN
- net USB_HUB/USB3DN_4_TXDM renamed USB_HUB/USB3DN_4_TXDN
- net USB_HUB/USB3UP_TXDM renamed USB_HUB/USB3UP_TXDN
Other:
- sheet USB_HUB ports: added USB2UP_DN, USB3DN_1_RXDN, USB3DN_1_TXDN, USB3DN_2_RXDN, USB3DN_2_TXDN, USB3DN_3_RXDN, USB3DN_3_TXDN, USB3DN_4_RXDN, USB3DN_4_TXDN, USB3UP_RXDN, USB3UP_TXDN; removed USB2UP_DM, USB3DN_1_RXDM, USB3DN_1_TXDM, USB3DN_2_RXDM, USB3DN_2_TXDM, USB3DN_3_RXDM, USB3DN_3_TXDM, USB3DN_4_RXDM, USB3DN_4_TXDM, USB3UP_RXDM, USB3UP_TXDM
- note added: "I_{in} = (V_{out} / (V_{in} * n)) * I_{out} 5V BUCK: I_{in} = (5 / (12 * 0.8)) * 8 I_{in} = 4.2A 1.15V BUCK: I_{in} = (1.15 / (12 * 0.8)) * 2.5 I_{in} = 0.3A Total I_{in} = 4.5A, Assume worst case from 3V3 and other sources, 5A"
- note added: "Max Current Consumption: 5V: 8A 3V: 400mA 1.15V: 2.5A"
- note removed: "Max Current Consumption: 5V: 13A 3V: 400mA 1.15V: 2.5A"

Commit message: Updates from the livestream
Connections:
- net UFP_MUX/TXn renamed TXN
- net UFP_MUX/TXp renamed TXP
Other:
- moved on the sheet: C5

Commit message: Updates from the livestream
Connections:
- net UFP_MUX/TX1n renamed TX1_N
- net UFP_MUX/TX1p renamed TX1_P
- net UFP_MUX/TX2n renamed TX2_N
- net UFP_MUX/TX2p renamed TX2_P
Other:
- moved on the sheet: C10, C11, C12, C13, C14, C5, C6, C7, C8, C9
