File: kicad_proj/mte_usb_hub/usb_a_filter.kicad_sch (KiCad schematic)
At the start: 5 parts

Commit message: Updates input protection, output BC enabled
Parts:
- gave numbers to parts that had none: 5
Connections:
- net GND_IN: no longer D2.9, D3.9
- net USB2_DN_IN: now also D3.6
- net USB2_DP_IN: now also D3.7
- net USB3_DN_RXDN_IN: now also D2.6, D2.9
- net USB3_DN_RXDP_IN: now also D2.10, D2.7
- net at D3.1: now also D3.10
- net at D3.2: now also D3.9
- no-connect marks 2 -> 0
Changed lines of the file:
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@@
-(kicad_sch (version 20210126) (generator eeschema)
+(kicad_sch (version 20210406) (generator eeschema)
   (paper "A4")
   (junction (at 66.04 114.3) (diameter 1.016) (color 0 0 0 0))
-  (junction (at 68.58 114.3) (diameter 1.016) (color 0 0 0 0))
-  (junction (at 78.74 114.3) (diameter 1.016) (color 0 0 0 0))
   (junction (at 81.28 114.3) (diameter 1.016) (color 0 0 0 0))
   (junction (at 82.55 114.3) (diameter 1.016) (color 0 0 0 0))
@@
   (junction (at 104.14 102.87) (diameter 1.016) (color 0 0 0 0))
   (junction (at 104.14 114.3) (diameter 1.016) (color 0 0 0 0))
-  (no_connect (at 83.82 105.41))
-  (no_connect (at 86.36 105.41))
   (wire (pts (xy 60.96 66.04) (xy 82.55 66.04))
     (stroke (width 0) (type solid) (color 0 0 0 0))
@@
     (stroke (width 0) (type solid) (color 0 0 0 0))
   )
-  (wire (pts (xy 66.04 114.3) (xy 68.58 114.3))
+  (wire (pts (xy 66.04 114.3) (xy 81.28 114.3))
     (stroke (width 0) (type solid) (color 0 0 0 0))
   )
@@
     (stroke (width 0) (type solid) (color 0 0 0 0))
   )
-  (wire (pts (xy 68.58 114.3) (xy 78.74 114.3))
-    (stroke (width 0) (type solid) (color 0 0 0 0))
-  )
   (wire (pts (xy 78.74 96.52) (xy 86.36 96.52))
     (stroke (width 0) (type solid) (color 0 0 0 0))
   )
   (wire (pts (xy 78.74 105.41) (xy 78.74 96.52))
-    (stroke (width 0) (type solid) (color 0 0 0 0))
-  )
-  (wire (pts (xy 78.74 114.3) (xy 81.28 114.3))
     (stroke (width 0) (type solid) (color 0 0 0 0))
   )
@@
   (symbol (lib_id "diodes:ESD9X3.3ST5G") (at 99.06 109.22 270)
     (in_bom yes) (on_board yes)
-    (property "Reference" "D?" (id 0) (at 99.6697 106.1656 90)
+    (property "Reference" "D4" (id 0) (at 99.6697 106.1656 90)
       (effects (font (size 1.27 1.27)) (justify left))
     )
@@
   (symbol (lib_id "capacitors:GRM21BR61H106ME43") (at 104.14 107.95 0)
     (in_bom yes) (on_board yes)
-    (property "Reference" "C?" (id 0) (at 104.5211 105.5306 0)
+    (property "Reference" "C73" (id 0) (at 104.5211 105.5306 0)
       (effects (font (size 1.27 1.27)) (justify left))
     )
@@
   (symbol (lib_id "capacitors:GRM21BR61H106ME43") (at 109.22 107.95 0)
     (in_bom yes) (on_board yes)
-    (property "Reference" "C?" (id 0) (at 109.6011 105.5306 0)
+    (property "Reference" "C74" (id 0) (at 109.6011 105.5306 0)
       (effects (font (size 1.27 1.27)) (justify left))
     )
@@
   (symbol (lib_id "mte_usb_hub:ESD8004MUTAG") (at 64.77 110.49 0)
     (in_bom yes) (on_board yes)
-    (property "Reference" "D?" (id 0) (at 70.4851 110.49 0)
+    (property "Reference" "D2" (id 0) (at 70.4851 110.49 0)
       (effects (font (size 1.27 1.27)) (justify left))
     )
@@
   (symbol (lib_id "mte_usb_hub:ESD8004MUTAG") (at 82.55 110.49 0) (mirror y)
     (in_bom yes) (on_board yes)
-    (property "Reference" "D?" (id 0) (at 76.8349 110.49 0)
-      (effects (font (size 1.27 1.27)) (justify left))
-    )
+    (property "Reference" "D3" (id 0) (at 76.8349 110.49 0)
+      (effects (font (size 1.27 1.27)) (justify left))
+    )

Commit message: New changes from the livestream
Starts the layout
Parts:
- C73, C74: footprint footprints:CAPACITOR_0805N -> mte_usb_footprints:CAPACITOR_0805N
- D2, D3: footprint (none) -> mte_usb_footprints:ESD8004MUTAG
- D4: footprint footprints:SODFL1006X43N -> mte_usb_footprints:SODFL1006X43N
Connections:
- net USB3_DN_RXDN_IN: no longer D2.5, D2.6
- net USB3_DN_RXDP_IN: no longer D2.4, D2.7
- new net USB3_DN_TXDN_IN: D2.5, D2.6
- new net USB3_DN_TXDP_IN: D2.4, D2.7
Changed lines of the file:
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@@
     (effects (font (size 1.27 1.27)) (justify right bottom))
   )
-  (label "USB3_TXDN" (at 60.96 101.6 180)
-    (effects (font (size 1.27 1.27)) (justify right bottom))
-  )
-  (label "USB3_TXDP" (at 60.96 104.14 180)
+  (label "USB3_RXDN" (at 60.96 101.6 180)
+    (effects (font (size 1.27 1.27)) (justify right bottom))
+  )
+  (label "USB3_RXDP" (at 60.96 104.14 180)
     (effects (font (size 1.27 1.27)) (justify right bottom))
   )
@@
     (effects (font (size 1.27 1.27)) (justify right bottom))
   )
-  (label "USB3_TXDN" (at 78.74 87.63 180)
-    (effects (font (size 1.27 1.27)) (justify right bottom))
-  )
-  (label "USB3_TXDP" (at 78.74 90.17 180)
+  (label "USB3_RXDN" (at 78.74 87.63 180)
+    (effects (font (size 1.27 1.27)) (justify right bottom))
+  )
+  (label "USB3_RXDP" (at 78.74 90.17 180)
     (effects (font (size 1.27 1.27)) (justify right bottom))
   )
@@
       (effects (font (size 1.27 1.27)) hide)
     )
-    (property "Footprint" "footprints:SODFL1006X43N" (id 2) (at 99.06 109.22 0)
+    (property "Footprint" "mte_usb_footprints:SODFL1006X43N" (id 2) (at 99.06 109.22 0)
       (effects (font (size 1.27 1.27)) hide)
     )
@@
       (effects (font (size 1.27 1.27)) (justify left) hide)
     )
-    (property "Footprint" "footprints:CAPACITOR_0805N" (id 2) (at 105.1052 111.76 0)
+    (property "Footprint" "mte_usb_footprints:CAPACITOR_0805N" (id 2) (at 105.1052 111.76 0)
       (effects (font (size 1.27 1.27)) hide)
     )
@@
       (effects (font (size 1.27 1.27)) (justify left) hide)
     )
-    (property "Footprint" "footprints:CAPACITOR_0805N" (id 2) (at 110.1852 111.76 0)
+    (property "Footprint" "mte_usb_footprints:CAPACITOR_0805N" (id 2) (at 110.1852 111.76 0)
       (effects (font (size 1.27 1.27)) hide)
     )
@@
       (effects (font (size 1.27 1.27)) hide)
     )
-    (property "Footprint" "" (id 2) (at 64.77 110.49 0)
+    (property "Footprint" "mte_usb_footprints:ESD8004MUTAG" (id 2) (at 64.77 110.49 0)
       (effects (font (size 1.27 1.27)) hide)
     )
@@
       (effects (font (size 1.27 1.27)) hide)
     )
-    (property "Footprint" "" (id 2) (at 82.55 110.49 0)
-      (effects (font (size 1.27 1.27)) hide)
-    )
+    (property "Footprint" "mte_usb_footprints:ESD8004MUTAG" (id 2) (at 82.55 110.49 0)
+      (effects (font (size 1.27 1.27)) hide)
+    )

Commit message: Updates from the livestream
Parts:
- renumbered C73 to C83, C74 to C84, D2 to D15, D3 to D16, D4 to D17
Connections:
- net USB3_DN_RXDN_IN: now also D15.1, D15.10; no longer D15.2, D15.9
- net USB3_DN_RXDP_IN: now also D15.2, D15.9; no longer D15.1, D15.10
- net USB3_DN_TXDN_IN: now also D15.4, D15.7; no longer D15.5, D15.6
- net USB3_DN_TXDP_IN: now also D15.5, D15.6; no longer D15.4, D15.7
Changed lines of the file:
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@@
-(kicad_sch (version 20210406) (generator eeschema)
+(kicad_sch (version 20210606) (generator eeschema)
   (paper "A4")
   (junction (at 66.04 114.3) (diameter 1.016) (color 0 0 0 0))
@@
     (stroke (width 0) (type solid) (color 0 0 0 0))
   )
-  (label "USB3_TXDN" (at 60.96 96.52 180)
-    (effects (font (size 1.27 1.27)) (justify right bottom))
-  )
-  (label "USB3_TXDP" (at 60.96 99.06 180)
-    (effects (font (size 1.27 1.27)) (justify right bottom))
-  )
-  (label "USB3_RXDN" (at 60.96 101.6 180)
-    (effects (font (size 1.27 1.27)) (justify right bottom))
-  )
-  (label "USB3_RXDP" (at 60.96 104.14 180)
+  (label "USB3_TXDP" (at 60.96 96.52 180)
+    (effects (font (size 1.27 1.27)) (justify right bottom))
+  )
+  (label "USB3_TXDN" (at 60.96 99.06 180)
+    (effects (font (size 1.27 1.27)) (justify right bottom))
+  )
+  (label "USB3_RXDP" (at 60.96 101.6 180)
+    (effects (font (size 1.27 1.27)) (justify right bottom))
+  )
+  (label "USB3_RXDN" (at 60.96 104.14 180)
     (effects (font (size 1.27 1.27)) (justify right bottom))
   )
@@
   (symbol (lib_id "diodes:ESD9X3.3ST5G") (at 99.06 109.22 270)
     (in_bom yes) (on_board yes)
-    (property "Reference" "D4" (id 0) (at 99.6697 106.1656 90)
+    (property "Reference" "D17" (id 0) (at 99.6697 106.1656 90)
       (effects (font (size 1.27 1.27)) (justify left))
     )
@@
   (symbol (lib_id "capacitors:GRM21BR61H106ME43") (at 104.14 107.95 0)
     (in_bom yes) (on_board yes)
-    (property "Reference" "C73" (id 0) (at 104.5211 105.5306 0)
+    (property "Reference" "C83" (id 0) (at 104.5211 105.5306 0)
       (effects (font (size 1.27 1.27)) (justify left))
     )
@@
   (symbol (lib_id "capacitors:GRM21BR61H106ME43") (at 109.22 107.95 0)
     (in_bom yes) (on_board yes)
-    (property "Reference" "C74" (id 0) (at 109.6011 105.5306 0)
+    (property "Reference" "C84" (id 0) (at 109.6011 105.5306 0)
       (effects (font (size 1.27 1.27)) (justify left))
     )
@@
   (symbol (lib_id "mte_usb_hub:ESD8004MUTAG") (at 64.77 110.49 0)
     (in_bom yes) (on_board yes)
-    (property "Reference" "D2" (id 0) (at 70.4851 110.49 0)
+    (property "Reference" "D15" (id 0) (at 70.4851 110.49 0)
       (effects (font (size 1.27 1.27)) (justify left))
     )
@@
   (symbol (lib_id "mte_usb_hub:ESD8004MUTAG") (at 82.55 110.49 0) (mirror y)
     (in_bom yes) (on_board yes)
-    (property "Reference" "D3" (id 0) (at 76.8349 110.49 0)
-      (effects (font (size 1.27 1.27)) (justify left))
-    )
+    (property "Reference" "D16" (id 0) (at 76.8349 110.49 0)
+      (effects (font (size 1.27 1.27)) (justify left))
+    )

Commit message: Updates from the livestream
Parts:
- renumbered C83 to C81, C84 to C82, D15 to D12, D16 to D13, D17 to D14
Changed lines of the file:
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@@
   (symbol (lib_id "diodes:ESD9X3.3ST5G") (at 99.06 109.22 270)
     (in_bom yes) (on_board yes)
-    (property "Reference" "D17" (id 0) (at 99.6697 106.1656 90)
+    (property "Reference" "D14" (id 0) (at 99.6697 106.1656 90)
       (effects (font (size 1.27 1.27)) (justify left))
     )
@@
   (symbol (lib_id "capacitors:GRM21BR61H106ME43") (at 104.14 107.95 0)
     (in_bom yes) (on_board yes)
-    (property "Reference" "C83" (id 0) (at 104.5211 105.5306 0)
+    (property "Reference" "C81" (id 0) (at 104.5211 105.5306 0)
       (effects (font (size 1.27 1.27)) (justify left))
     )
@@
   (symbol (lib_id "capacitors:GRM21BR61H106ME43") (at 109.22 107.95 0)
     (in_bom yes) (on_board yes)
-    (property "Reference" "C84" (id 0) (at 109.6011 105.5306 0)
+    (property "Reference" "C82" (id 0) (at 109.6011 105.5306 0)
       (effects (font (size 1.27 1.27)) (justify left))
     )
@@
   (symbol (lib_id "mte_usb_hub:ESD8004MUTAG") (at 64.77 110.49 0)
     (in_bom yes) (on_board yes)
-    (property "Reference" "D15" (id 0) (at 70.4851 110.49 0)
+    (property "Reference" "D12" (id 0) (at 70.4851 110.49 0)
       (effects (font (size 1.27 1.27)) (justify left))
     )
@@
   (symbol (lib_id "mte_usb_hub:ESD8004MUTAG") (at 82.55 110.49 0) (mirror y)
     (in_bom yes) (on_board yes)
-    (property "Reference" "D16" (id 0) (at 76.8349 110.49 0)
+    (property "Reference" "D13" (id 0) (at 76.8349 110.49 0)
       (effects (font (size 1.27 1.27)) (justify left))
     )

Commit message: Livestream updates
Parts:
- renumbered C81 to C79, C82 to C80, D13 to D10, D14 to D11, D12 to D9
Connections:
- no-connect marks 0 -> 2
Changed lines of the file:
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@@
   (junction (at 104.14 102.87) (diameter 1.016) (color 0 0 0 0))
   (junction (at 104.14 114.3) (diameter 1.016) (color 0 0 0 0))
+  (no_connect (at 83.82 105.41))
+  (no_connect (at 86.36 105.41))
   (wire (pts (xy 60.96 66.04) (xy 82.55 66.04))
     (stroke (width 0) (type solid) (color 0 0 0 0))
@@
   (symbol (lib_id "diodes:ESD9X3.3ST5G") (at 99.06 109.22 270)
     (in_bom yes) (on_board yes)
-    (property "Reference" "D14" (id 0) (at 99.6697 106.1656 90)
+    (property "Reference" "D11" (id 0) (at 99.6697 106.1656 90)
       (effects (font (size 1.27 1.27)) (justify left))
     )
@@
   (symbol (lib_id "capacitors:GRM21BR61H106ME43") (at 104.14 107.95 0)
     (in_bom yes) (on_board yes)
-    (property "Reference" "C81" (id 0) (at 104.5211 105.5306 0)
+    (property "Reference" "C79" (id 0) (at 104.5211 105.5306 0)
       (effects (font (size 1.27 1.27)) (justify left))
     )
@@
   (symbol (lib_id "capacitors:GRM21BR61H106ME43") (at 109.22 107.95 0)
     (in_bom yes) (on_board yes)
-    (property "Reference" "C82" (id 0) (at 109.6011 105.5306 0)
+    (property "Reference" "C80" (id 0) (at 109.6011 105.5306 0)
       (effects (font (size 1.27 1.27)) (justify left))
     )
@@
   (symbol (lib_id "mte_usb_hub:ESD8004MUTAG") (at 64.77 110.49 0)
     (in_bom yes) (on_board yes)
-    (property "Reference" "D12" (id 0) (at 70.4851 110.49 0)
+    (property "Reference" "D9" (id 0) (at 70.4851 110.49 0)
       (effects (font (size 1.27 1.27)) (justify left))
     )
@@
   (symbol (lib_id "mte_usb_hub:ESD8004MUTAG") (at 82.55 110.49 0) (mirror y)
     (in_bom yes) (on_board yes)
-    (property "Reference" "D13" (id 0) (at 76.8349 110.49 0)
-      (effects (font (size 1.27 1.27)) (justify left))
-    )
+    (property "Reference" "D10" (id 0) (at 76.8349 110.49 0)
+      (effects (font (size 1.27 1.27)) (justify left))
+    )
