File: kicad_proj/mte_usb_hub/usb_c_filter.kicad_sch (KiCad schematic)
At the start: 6 parts

Commit message: New changes from the livestream
Starts the layout
Parts:
- C75, C76: footprint footprints:CAPACITOR_0402N -> mte_usb_footprints:CAPACITOR_0402N
- D5, D6, D7: footprint (none) -> mte_usb_footprints:ESD8004MUTAG
- D8: footprint footprints:SODFL1006X43N -> mte_usb_footprints:SODFL1006X43N
Other:
- moved on the sheet: D7
Changed lines of the file:
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@@
     (stroke (width 0) (type solid) (color 0 0 0 0))
   )
-  (wire (pts (xy 102.87 93.98) (xy 113.03 93.98))
-    (stroke (width 0) (type solid) (color 0 0 0 0))
-  )
-  (wire (pts (xy 102.87 99.06) (xy 107.95 99.06))
-    (stroke (width 0) (type solid) (color 0 0 0 0))
-  )
-  (wire (pts (xy 105.41 101.6) (xy 102.87 101.6))
-    (stroke (width 0) (type solid) (color 0 0 0 0))
-  )
-  (wire (pts (xy 105.41 102.87) (xy 105.41 101.6))
-    (stroke (width 0) (type solid) (color 0 0 0 0))
-  )
-  (wire (pts (xy 107.95 99.06) (xy 107.95 102.87))
+  (wire (pts (xy 102.87 92.71) (xy 113.03 92.71))
+    (stroke (width 0) (type solid) (color 0 0 0 0))
+  )
+  (wire (pts (xy 102.87 97.79) (xy 107.95 97.79))
+    (stroke (width 0) (type solid) (color 0 0 0 0))
+  )
+  (wire (pts (xy 105.41 100.33) (xy 102.87 100.33))
+    (stroke (width 0) (type solid) (color 0 0 0 0))
+  )
+  (wire (pts (xy 105.41 101.6) (xy 105.41 100.33))
+    (stroke (width 0) (type solid) (color 0 0 0 0))
+  )
+  (wire (pts (xy 107.95 97.79) (xy 107.95 101.6))
+    (stroke (width 0) (type solid) (color 0 0 0 0))
+  )
+  (wire (pts (xy 107.95 109.22) (xy 107.95 110.49))
     (stroke (width 0) (type solid) (color 0 0 0 0))
   )
@@
     (stroke (width 0) (type solid) (color 0 0 0 0))
   )
-  (wire (pts (xy 110.49 96.52) (xy 102.87 96.52))
-    (stroke (width 0) (type solid) (color 0 0 0 0))
-  )
-  (wire (pts (xy 110.49 102.87) (xy 110.49 96.52))
-    (stroke (width 0) (type solid) (color 0 0 0 0))
-  )
-  (wire (pts (xy 113.03 93.98) (xy 113.03 102.87))
+  (wire (pts (xy 110.49 95.25) (xy 102.87 95.25))
+    (stroke (width 0) (type solid) (color 0 0 0 0))
+  )
+  (wire (pts (xy 110.49 101.6) (xy 110.49 95.25))
+    (stroke (width 0) (type solid) (color 0 0 0 0))
+  )
+  (wire (pts (xy 110.49 109.22) (xy 110.49 110.49))
+    (stroke (width 0) (type solid) (color 0 0 0 0))
+  )
+  (wire (pts (xy 110.49 110.49) (xy 127 110.49))
+    (stroke (width 0) (type solid) (color 0 0 0 0))
+  )
+  (wire (pts (xy 113.03 92.71) (xy 113.03 101.6))
     (stroke (width 0) (type solid) (color 0 0 0 0))
   )
@@
     (stroke (width 0) (type solid) (color 0 0 0 0))
   )
-  (wire (pts (xy 127 110.49) (xy 110.49 110.49))
-    (stroke (width 0) (type solid) (color 0 0 0 0))
-  )
   (wire (pts (xy 133.35 96.52) (xy 133.35 99.06))
     (stroke (width 0) (type solid) (color 0 0 0 0))
@@
     (effects (font (size 1.27 1.27)) (justify left bottom))
   )
-  (label "CC1" (at 102.87 93.98 0)
-    (effects (font (size 1.27 1.27)) (justify left bottom))
-  )
-  (label "CC2" (at 102.87 96.52 0)
-    (effects (font (size 1.27 1.27)) (justify left bottom))
-  )
-  (label "D+" (at 102.87 99.06 0)
-    (effects (font (size 1.27 1.27)) (justify left bottom))
-  )
-  (label "D-" (at 102.87 101.6 0)
+  (label "CC1" (at 102.87 92.71 0)
+    (effects (font (size 1.27 1.27)) (justify left bottom))
+  )
+  (label "CC2" (at 102.87 95.25 0)
+    (effects (font (size 1.27 1.27)) (justify left bottom))
+  )
+  (label "D+" (at 102.87 97.79 0)
+    (effects (font (size 1.27 1.27)) (justify left bottom))
+  )
+  (label "D-" (at 102.87 100.33 0)
     (effects (font (size 1.27 1.27)) (justify left bottom))
   )
@@
       (effects (font (size 1.27 1.27)) hide)
     )
-    (property "Footprint" "footprints:SODFL1006X43N" (id 2) (at 127 102.87 0)
+    (property "Footprint" "mte_usb_footprints:SODFL1006X43N" (id 2) (at 127 102.87 0)
       (effects (font (size 1.27 1.27)) hide)
     )
@@
       (effects (font (size 1.27 1.27)) (justify left) hide)
     )
-    (property "Footprint" "footprints:CAPACITOR_0402N" (id 2) (at 134.3152 106.68 0)
+    (property "Footprint" "mte_usb_footprints:CAPACITOR_0402N" (id 2) (at 134.3152 106.68 0)
       (effects (font (size 1.27 1.27)) hide)
     )
@@
       (effects (font (size 1.27 1.27)) (justify left) hide)
     )
-    (property "Footprint" "footprints:CAPACITOR_0402N" (id 2) (at 140.6652 106.68 0)
+    (property "Footprint" "mte_usb_footprints:CAPACITOR_0402N" (id 2) (at 140.6652 106.68 0)
       (effects (font (size 1.27 1.27)) hide)
     )
@@
       (effects (font (size 1.27 1.27)) hide)
     )
-    (property "Footprint" "" (id 2) (at 76.2 106.68 0)
+    (property "Footprint" "mte_usb_footprints:ESD8004MUTAG" (id 2) (at 76.2 106.68 0)
       (effects (font (size 1.27 1.27)) hide)
     )
@@
       (effects (font (size 1.27 1.27)) hide)
     )
-    (property "Footprint" "" (id 2) (at 93.98 106.68 0)
+    (property "Footprint" "mte_usb_footprints:ESD8004MUTAG" (id 2) (at 93.98 106.68 0)
       (effects (font (size 1.27 1.27)) hide)
     )
@@
     (pin "9")
   )
-  (symbol (lib_id "mte_usb_hub:ESD8004MUTAG") (at 109.22 107.95 0) (mirror y) (unit 1)
-    (in_bom yes) (on_board yes)
-    (property "Reference" "D7" (id 0) (at 103.5049 107.95 0)
-      (effects (font (size 1.27 1.27)) (justify left))
-    )
-    (property "Value" "ESD8004MUTAG" (id 1) (at 109.22 107.95 0)
-      (effects (font (size 1.27 1.27)) hide)
-    )
-    (property "Footprint" "" (id 2) (at 109.22 107.95 0)
-      (effects (font (size 1.27 1.27)) hide)
-    )
-    (property "Datasheet" "" (id 3) (at 109.22 107.95 0)
-      (effects (font (size 1.27 1.27)) hide)
-    )
-    (property "id" "ESD8004MUTAG" (id 4) (at 109.22 107.95 0)
-      (effects (font (size 1.27 1.27)) hide)
-    )
-    (property "manf" "ON Semiconductor" (id 5) (at 109.22 107.95 0)
-      (effects (font (size 1.27 1.27)) hide)
-    )
+  (symbol (lib_id "mte_usb_hub:ESD8004MUTAG") (at 109.22 106.68 0) (mirror y) (unit 1)
+    (in_bom yes) (on_board yes)
+    (property "Reference" "D7" (id 0) (at 103.5049 106.68 0)
+      (effects (font (size 1.27 1.27)) (justify left))
+    )
+    (property "Value" "ESD8004MUTAG" (id 1) (at 109.22 106.68 0)
+      (effects (font (size 1.27 1.27)) hide)
+    )
+    (property "Footprint" "mte_usb_footprints:ESD8004MUTAG" (id 2) (at 109.22 106.68 0)
+      (effects (font (size 1.27 1.27)) hide)
+    )
+    (property "Datasheet" "" (id 3) (at 109.22 106.68 0)
+      (effects (font (size 1.27 1.27)) hide)
+    )
+    (property "id" "ESD8004MUTAG" (id 4) (at 109.22 106.68 0)
+      (effects (font (size 1.27 1.27)) hide)
+    )
+    (property "manf" "ON Semiconductor" (id 5) (at 109.22 106.68 0)
+      (effects (font (size 1.27 1.27)) hide)
+    )

Commit message: Updates from the livestream
Connections:
- net RX2+_IN: now also D6.1, D6.10; no longer D6.2, D6.9
- net RX2-_IN: now also D6.2, D6.9; no longer D6.1, D6.10
- net TX2+_IN: now also D6.4, D6.7; no longer D6.5, D6.6
- net TX2-_IN: now also D6.5, D6.6; no longer D6.4, D6.7
Changed lines of the file:
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@@
     (stroke (width 0) (type solid) (color 0 0 0 0))
   )
-  (label "RX1-" (at 67.31 92.71 0)
+  (label "_RX1-" (at 67.31 92.71 0)
     (effects (font (size 1.27 1.27)) (justify left bottom))
   )
-  (label "RX1+" (at 67.31 95.25 0)
+  (label "_RX1+" (at 67.31 95.25 0)
     (effects (font (size 1.27 1.27)) (justify left bottom))
   )
-  (label "TX1-" (at 67.31 97.79 0)
+  (label "_TX1-" (at 67.31 97.79 0)
     (effects (font (size 1.27 1.27)) (justify left bottom))
   )
-  (label "TX1+" (at 67.31 100.33 0)
+  (label "_TX1+" (at 67.31 100.33 0)
     (effects (font (size 1.27 1.27)) (justify left bottom))
   )
-  (label "RX2-" (at 85.09 92.71 0)
+  (label "_RX2+" (at 85.09 92.71 0)
     (effects (font (size 1.27 1.27)) (justify left bottom))
   )
-  (label "RX2+" (at 85.09 95.25 0)
+  (label "_RX2-" (at 85.09 95.25 0)
     (effects (font (size 1.27 1.27)) (justify left bottom))
   )
-  (label "TX2-" (at 85.09 97.79 0)
+  (label "_TX2+" (at 85.09 97.79 0)
     (effects (font (size 1.27 1.27)) (justify left bottom))
   )
-  (label "TX2+" (at 85.09 100.33 0)
+  (label "_TX2-" (at 85.09 100.33 0)
     (effects (font (size 1.27 1.27)) (justify left bottom))
   )
@@
     (effects (font (size 1.27 1.27)) (justify left bottom))
   )
-  (label "TX1+" (at 87.63 43.18 0)
+  (label "_TX1+" (at 87.63 43.18 0)
     (effects (font (size 1.27 1.27)) (justify left bottom))
   )
-  (label "TX1-" (at 87.63 45.72 0)
+  (label "_TX1-" (at 87.63 45.72 0)
     (effects (font (size 1.27 1.27)) (justify left bottom))
   )
-  (label "RX1+" (at 87.63 49.53 0)
+  (label "_RX1+" (at 87.63 49.53 0)
     (effects (font (size 1.27 1.27)) (justify left bottom))
   )
-  (label "RX1-" (at 87.63 52.07 0)
+  (label "_RX1-" (at 87.63 52.07 0)
     (effects (font (size 1.27 1.27)) (justify left bottom))
   )
-  (label "TX2+" (at 87.63 55.88 0)
+  (label "_TX2+" (at 87.63 55.88 0)
     (effects (font (size 1.27 1.27)) (justify left bottom))
   )
-  (label "TX2-" (at 87.63 58.42 0)
+  (label "_TX2-" (at 87.63 58.42 0)
     (effects (font (size 1.27 1.27)) (justify left bottom))
   )
-  (label "RX2+" (at 87.63 62.23 0)
+  (label "_RX2+" (at 87.63 62.23 0)
     (effects (font (size 1.27 1.27)) (justify left bottom))
   )
-  (label "RX2-" (at 87.63 64.77 0)
+  (label "_RX2-" (at 87.63 64.77 0)
     (effects (font (size 1.27 1.27)) (justify left bottom))
   )
@@
     (effects (font (size 1.27 1.27)) (justify left bottom))
   )
-  (label "D+" (at 87.63 74.93 0)
+  (label "_D+" (at 87.63 74.93 0)
     (effects (font (size 1.27 1.27)) (justify left bottom))
   )
-  (label "D-" (at 87.63 77.47 0)
+  (label "_D-" (at 87.63 77.47 0)
     (effects (font (size 1.27 1.27)) (justify left bottom))
   )
@@
     (effects (font (size 1.27 1.27)) (justify left bottom))
   )
-  (label "D+" (at 102.87 97.79 0)
+  (label "_D+" (at 102.87 97.79 0)
     (effects (font (size 1.27 1.27)) (justify left bottom))
   )
-  (label "D-" (at 102.87 100.33 0)
+  (label "_D-" (at 102.87 100.33 0)
     (effects (font (size 1.27 1.27)) (justify left bottom))
   )

Commit message: Livestream updates
Connections:
- net D+_IN: now also D7.5, D7.6; no longer D7.4, D7.7
- net D-_IN: now also D7.4, D7.7; no longer D7.5, D7.6
- net RX2+_IN: now also D6.4, D6.7; no longer D6.1, D6.10
- net RX2-_IN: now also D6.5, D6.6; no longer D6.2, D6.9
- net TX1+_IN: now also D5.2, D5.9; no longer D5.1, D5.10
- net TX1-_IN: now also D5.1, D5.10; no longer D5.2, D5.9
- net TX2+_IN: now also D6.1, D6.10; no longer D6.4, D6.7
- net TX2-_IN: now also D6.2, D6.9; no longer D6.5, D6.6
Changed lines of the file:
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@@
     (effects (font (size 1.27 1.27)) (justify left bottom))
   )
-  (label "_TX1-" (at 67.31 97.79 0)
+  (label "_TX1+" (at 67.31 97.79 0)
     (effects (font (size 1.27 1.27)) (justify left bottom))
   )
-  (label "_TX1+" (at 67.31 100.33 0)
+  (label "_TX1-" (at 67.31 100.33 0)
     (effects (font (size 1.27 1.27)) (justify left bottom))
   )
-  (label "_RX2+" (at 85.09 92.71 0)
+  (label "_TX2+" (at 85.09 92.71 0)
     (effects (font (size 1.27 1.27)) (justify left bottom))
   )
-  (label "_RX2-" (at 85.09 95.25 0)
+  (label "_TX2-" (at 85.09 95.25 0)
     (effects (font (size 1.27 1.27)) (justify left bottom))
   )
-  (label "_TX2+" (at 85.09 97.79 0)
+  (label "_RX2+" (at 85.09 97.79 0)
     (effects (font (size 1.27 1.27)) (justify left bottom))
   )
-  (label "_TX2-" (at 85.09 100.33 0)
+  (label "_RX2-" (at 85.09 100.33 0)
     (effects (font (size 1.27 1.27)) (justify left bottom))
   )
@@
     (effects (font (size 1.27 1.27)) (justify left bottom))
   )
-  (label "_D+" (at 102.87 97.79 0)
+  (label "_D-" (at 102.87 97.79 0)
     (effects (font (size 1.27 1.27)) (justify left bottom))
   )
-  (label "_D-" (at 102.87 100.33 0)
+  (label "_D+" (at 102.87 100.33 0)
     (effects (font (size 1.27 1.27)) (justify left bottom))
   )
